File: src/Power.sch (KiCad schematic (older format))
At the start: 14 parts, among them J1 USB, P1 CONN_2X2, U1 LP5907

Commit message: Approximately done.
Parts:
- removed J1: USB, symbol USB
- added J1, J2: CONN_5, symbol CONN_5
Connections:
- wire segments 41 -> 44
Changed lines of the file:
@@
 Sheet 2 2
 Title ""
-Date "1 aug 2014"
+Date "2 aug 2014"
 Rev ""
 Comp ""
@@
 Comment4 ""
 $EndDescr
-$Comp
-L USB J1
-U 1 1 53DBAF85
-P 7200 2000
-F 0 "J1" H 7150 2400 60  0000 C CNN
-F 1 "USB" V 6950 2150 60  0000 C CNN
-F 2 "" H 7200 2000 60  0000 C CNN
-F 3 "" H 7200 2000 60  0000 C CNN
-	1    7200 2000
-	1    0    0    -1
-$EndComp
-Text Label 6350 2200 0    60   ~ 0
-USB_5V
-Wire Wire Line
-	6250 2200 6800 2200
-$Comp
-L GND #PWR08
+Text Label 5850 1600 0    60   ~ 0
+USB_5V
+Wire Wire Line
+	5750 1600 6300 1600
+$Comp
+L GND #PWR09
 U 1 1 53DBAF95
-P 6700 2550
-F 0 "#PWR08" H 6700 2550 30  0001 C CNN
-F 1 "GND" H 6700 2480 30  0001 C CNN
-F 2 "" H 6700 2550 60  0000 C CNN
-F 3 "" H 6700 2550 60  0000 C CNN
-	1    6700 2550
-	1    0    0    -1
-$EndComp
-Wire Wire Line
-	6700 2550 6700 2350
-Wire Wire Line
-	6700 2350 6800 2350
+P 6200 2200
+F 0 "#PWR09" H 6200 2200 30  0001 C CNN
+F 1 "GND" H 6200 2130 30  0001 C CNN
+F 2 "" H 6200 2200 60  0000 C CNN
+F 3 "" H 6200 2200 60  0000 C CNN
+	1    6200 2200
+	1    0    0    -1
+$EndComp
+Wire Wire Line
+	6200 2200 6200 2000
+Wire Wire Line
+	6200 2000 6300 2000
 $Comp
 L LP5907 U1
@@
 USB_5V
 $Comp
-L GND #PWR09
+L GND #PWR010
 U 1 1 53DBB041
 P 6650 3850
-F 0 "#PWR09" H 6650 3850 30  0001 C CNN
+F 0 "#PWR010" H 6650 3850 30  0001 C CNN
 F 1 "GND" H 6650 3780 30  0001 C CNN
 F 2 "" H 6650 3850 60  0000 C CNN
@@
 	1    0    0    -1
 $EndComp
-Text Label 6550 2900 0    60   ~ 0
-USB_5V
+Text Label 6550 3000 0    60   ~ 0
+USB_5V
+Wire Wire Line
+	6250 3000 7000 3000
+Text Label 6400 2900 0    60   ~ 0
+Filtered_Vcc
 Wire Wire Line
 	6250 2900 7000 2900
-Text Label 6400 3000 0    60   ~ 0
-Filtered_Vcc
-Wire Wire Line
-	6250 3000 7000 3000
 Text Label 7950 2900 0    60   ~ 0
 Vcc
@@
 USB_5V
 Wire Wire Line
-	1800 1900 2900 1900
+	1800 1900 3200 1900
 Wire Wire Line
 	2300 1900 2300 2000
@@
 Connection ~ 2600 1900
 $Comp
-L GND #PWR010
+L GND #PWR011
 U 1 1 53DBD760
 P 2150 2550
-F 0 "#PWR010" H 2150 2550 30  0001 C CNN
+F 0 "#PWR011" H 2150 2550 30  0001 C CNN
 F 1 "GND" H 2150 2480 30  0001 C CNN
 F 2 "" H 2150 2550 60  0000 C CNN
@@
 	2150 2550 2150 2500
 Wire Wire Line
-	2150 2500 2900 2500
+	2150 2500 3200 2500
 Wire Wire Line
 	2900 2500 2900 2400
@@
 	2300 2400 2300 2500
 Connection ~ 2300 2500
-$Comp
-L CAPAPOL C13
-U 1 1 53DBD7BB
-P 1600 3400
-F 0 "C13" H 1650 3500 40  0000 L CNN
-F 1 "CAPAPOL" H 1650 3300 40  0000 L CNN
-F 2 "~" H 1700 3250 30  0000 C CNN
-F 3 "~" H 1600 3400 300 0000 C CNN
-	1    1600 3400
-	1    0    0    -1
-$EndComp
 $Comp
 L CAPAPOL C14
@@
 	1100 3100 3400 3100
 Wire Wire Line
-	1600 3100 1600 3200
-Wire Wire Line
 	1900 3100 1900 3200
-Connection ~ 1600 3100
 Wire Wire Line
 	2200 3100 2200 3200
 Connection ~ 1900 3100
 $Comp
-L GND #PWR011
+L GND #PWR012
 U 1 1 53DBD7D4
 P 1450 3750
-F 0 "#PWR011" H 1450 3750 30  0001 C CNN
+F 0 "#PWR012" H 1450 3750 30  0001 C CNN
 F 1 "GND" H 1450 3680 30  0001 C CNN
 F 2 "" H 1450 3750 60  0000 C CNN
@@
 	1900 3600 1900 3700
 Connection ~ 1900 3700
-Wire Wire Line
-	1600 3600 1600 3700
-Connection ~ 1600 3700
 $Comp
 L CAPAPOL C16
@@
 	3400 3700 3400 3600
 Connection ~ 3100 3700
+$Comp
+L CONN_5 J1
+U 1 1 53DC815D
+P 6700 1800
+F 0 "J1" V 6650 1800 50  0000 C CNN
+F 1 "CONN_5" V 6750 1800 50  0000 C CNN
+F 2 "" H 6700 1800 60  0000 C CNN
+F 3 "" H 6700 1800 60  0000 C CNN
+	1    6700 1800
+	1    0    0    -1
+$EndComp
+Text Label 7050 1600 0    60   ~ 0
+USB_5V
+Wire Wire Line
+	6950 1600 7500 1600
+$Comp
+L GND #PWR013
+U 1 1 53DC8189
+P 7400 2200
+F 0 "#PWR013" H 7400 2200 30  0001 C CNN
+F 1 "GND" H 7400 2130 30  0001 C CNN
+F 2 "" H 7400 2200 60  0000 C CNN
+F 3 "" H 7400 2200 60  0000 C CNN
+	1    7400 2200
+	1    0    0    -1
+$EndComp
+Wire Wire Line
+	7400 2200 7400 2000
+Wire Wire Line
+	7400 2000 7500 2000
+$Comp
+L CONN_5 J2
+U 1 1 53DC8191
+P 7900 1800
+F 0 "J2" V 7850 1800 50  0000 C CNN
+F 1 "CONN_5" V 7950 1800 50  0000 C CNN
+F 2 "" H 7900 1800 60  0000 C CNN
+F 3 "" H 7900 1800 60  0000 C CNN
+	1    7900 1800
+	1    0    0    -1
+$EndComp
+$Comp
+L CAPAPOL C13
+U 1 1 53DCF18A
+P 3200 2200
+F 0 "C13" H 3250 2300 40  0000 L CNN
+F 1 "CAPAPOL" H 3250 2100 40  0000 L CNN
+F 2 "~" H 3300 2050 30  0000 C CNN
+F 3 "~" H 3200 2200 300 0000 C CNN
+	1    3200 2200
+	1    0    0    -1
+$EndComp
+Wire Wire Line
+	3200 1900 3200 2000
+Connection ~ 2900 1900
+Wire Wire Line
+	3200 2500 3200 2400
+Connection ~ 2900 2500
 $EndSCHEMATC
