File: src/MonoAudioSharingAmp.sch (KiCad schematic (older format))
At the start: 33 parts, among them K2 CONN_3, K3 CONN_3, K4 CONN_3, P2 CONN_2X2, U2 DUAL_OPAMP, U3 DUAL_OPAMP, U4 DUAL_OPAMP, U5 DUAL_OPAMP

Commit message: Approximately done.
Parts:
- removed K2, K3, K4: CONN_3, symbol CONN_3
- added K2, K3, K4: CONN_5, symbol CONN_5
- added R12: R, ~, symbol R
- gave numbers to parts that had none: 1
Connections:
- net labels removed: CENTERD_INPUT
- wire segments 195 -> 162
Other:
- moved on the sheet: C1, C2, C3, P2

Commit message: Added mounting hole. Added text messages. Enlarged the board.
Parts:
- added C4: CAPAPOL, ~, symbol CAPAPOL
- added H1, H2, H3, H4, P3, P4, P5: CONN_1, symbol CONN_1
Connections:
- wire segments 162 -> 168
Changed lines of the file:
@@
 $EndComp
 Wire Wire Line
-	2250 1450 4100 1450
+	2250 1450 4400 1450
 Wire Wire Line
 	2500 1450 2500 1600
@@
 Connection ~ 3400 1450
 Wire Wire Line
-	2250 2100 3700 2100
+	2250 2100 4000 2100
 Wire Wire Line
 	2500 2100 2500 2000
@@
 	3700 2100 3700 2000
 Connection ~ 3400 2100
-Text Label 3800 1450 0    60   ~ 0
+Text Label 4100 1450 0    60   ~ 0
 VGND
 Connection ~ 3700 1450
@@
 	1    0    0    -1
 $EndComp
-$Comp
-L GND #PWR08
-U 1 1 53DC89CF
-P 4350 3350
-F 0 "#PWR08" H 4350 3350 30  0001 C CNN
-F 1 "GND" H 4350 3280 30  0001 C CNN
-F 2 "" H 4350 3350 60  0000 C CNN
-F 3 "" H 4350 3350 60  0000 C CNN
-	1    4350 3350
-	1    0    0    -1
-$EndComp
 Wire Wire Line
 	4350 3350 4350 3250
@@
 	4350 2750 4350 2650
 Connection ~ 4350 2650
+$Comp
+L CONN_1 H1
+U 1 1 53DD1725
+P 8550 950
+F 0 "H1" H 8630 950 40  0000 L CNN
+F 1 "CONN_1" H 8550 1005 30  0001 C CNN
+F 2 "" H 8550 950 60  0000 C CNN
+F 3 "" H 8550 950 60  0000 C CNN
+	1    8550 950
+	1    0    0    -1
+$EndComp
+$Comp
+L CONN_1 H2
+U 1 1 53DD1740
+P 8550 1050
+F 0 "H2" H 8630 1050 40  0000 L CNN
+F 1 "CONN_1" H 8550 1105 30  0001 C CNN
+F 2 "" H 8550 1050 60  0000 C CNN
+F 3 "" H 8550 1050 60  0000 C CNN
+	1    8550 1050
+	1    0    0    -1
+$EndComp
+$Comp
+L CONN_1 H3
+U 1 1 53DD174F
+P 8550 1150
+F 0 "H3" H 8630 1150 40  0000 L CNN
+F 1 "CONN_1" H 8550 1205 30  0001 C CNN
+F 2 "" H 8550 1150 60  0000 C CNN
+F 3 "" H 8550 1150 60  0000 C CNN
+	1    8550 1150
+	1    0    0    -1
+$EndComp
+$Comp
+L CONN_1 H4
+U 1 1 53DD1770
+P 8550 1250
+F 0 "H4" H 8630 1250 40  0000 L CNN
+F 1 "CONN_1" H 8550 1305 30  0001 C CNN
+F 2 "" H 8550 1250 60  0000 C CNN
+F 3 "" H 8550 1250 60  0000 C CNN
+	1    8550 1250
+	1    0    0    -1
+$EndComp
+Text Label 4450 3350 0    60   ~ 0
+VGND
+Wire Wire Line
+	4350 3350 4900 3350
+$Comp
+L CONN_1 P3
+U 1 1 53DD277E
+P 4550 1450
+F 0 "P3" H 4630 1450 40  0000 L CNN
+F 1 "CONN_1" H 4550 1505 30  0001 C CNN
+F 2 "" H 4550 1450 60  0000 C CNN
+F 3 "" H 4550 1450 60  0000 C CNN
+	1    4550 1450
+	1    0    0    -1
+$EndComp
+$Comp
+L CONN_1 P4
+U 1 1 53DD27A5
+P 6850 1600
+F 0 "P4" H 6930 1600 40  0000 L CNN
+F 1 "CONN_1" H 6850 1655 30  0001 C CNN
+F 2 "" H 6850 1600 60  0000 C CNN
+F 3 "" H 6850 1600 60  0000 C CNN
+	1    6850 1600
+	1    0    0    -1
+$EndComp
+$Comp
+L CONN_1 P5
+U 1 1 53DD27BD
+P 6850 1700
+F 0 "P5" H 6930 1700 40  0000 L CNN
+F 1 "CONN_1" H 6850 1755 30  0001 C CNN
+F 2 "" H 6850 1700 60  0000 C CNN
+F 3 "" H 6850 1700 60  0000 C CNN
+	1    6850 1700
+	1    0    0    -1
+$EndComp
+$Comp
+L GND #PWR08
+U 1 1 53DD27CC
+P 6600 1800
+F 0 "#PWR08" H 6600 1800 30  0001 C CNN
+F 1 "GND" H 6600 1730 30  0001 C CNN
+F 2 "" H 6600 1800 60  0000 C CNN
+F 3 "" H 6600 1800 60  0000 C CNN
+	1    6600 1800
+	1    0    0    -1
+$EndComp
+Wire Wire Line
+	6600 1600 6600 1800
+Wire Wire Line
+	6600 1700 6700 1700
+Wire Wire Line
+	6700 1600 6600 1600
+Connection ~ 6600 1700
+$Comp
+L CAPAPOL C4
+U 1 1 53DD2C1B
+P 4000 1800
+F 0 "C4" H 4050 1900 40  0000 L CNN
+F 1 "CAPAPOL" H 4050 1700 40  0000 L CNN
+F 2 "~" H 4100 1650 30  0000 C CNN
+F 3 "~" H 4000 1800 300 0000 C CNN
+	1    4000 1800
+	1    0    0    -1
+$EndComp
+Wire Wire Line
+	4000 1600 4000 1450
+Connection ~ 4000 1450
+Wire Wire Line
+	4000 2100 4000 2000
+Connection ~ 3700 2100
 $EndSCHEMATC
